Commit message: One (1) working joint

File: turtle_brick/urdf/turtle_bot.urdf (robot description, URDF)
Before this commit: robot turtlebot, 2 links, 1 joints
Links:
- added link pillar_link; visual cylinder length=1 radius=0.1
- added link platform_link; visual cylinder length=.1 radius=1
Joints:
- added joint pillar_joint: type fixed, parent base_link, child pillar_link, origin xyz=0 0 .25 rpy=0 0 0
- added joint platform_joint: type revolute, parent pillar_link, child platform_link, origin xyz=0 0 1.05 rpy=0 0 0, axis 0 1 0, limit lower=0 upper=0.7853981633974483 effort=100 velocity=100
- joint base_joint: origin xyz=0 0 1 rpy=0 0 0 -> xyz=0 0 0 rpy=0 0 0

File: turtle_brick/urdf/turtle_bot.urdf.xacro (robot description, xacro)
@@ -2,9 +2,10 @@
 <robot xmlns:xacro="http://www.ros.org/wiki/xacro"  name="turtlebot">
     <xacro:include filename="usefulstuff.xacro" />
-    <xacro:property name="stem_length" value="1" />
+    <xacro:property name="platform_height" value="1" />
+    <xacro:property name="platform_radius" value="1" />
     <xacro:property name="wheel_radius" value="0.5" />
     <link name="world"></link>
     <joint name="base_joint" type="fixed">
-        <origin xyz="0 0 1" rpy="0 0 0"/>
+        <origin xyz="0 0 0" rpy="0 0 0"/>
         <parent link="world"/>
         <child link="base_link"/>
@@ -19,12 +20,48 @@
         </visual>
     </link>
-    <link name="stem_link">
+    <joint name="pillar_joint" type="fixed">
+        <origin xyz="0 0 .25" rpy="0 0 0"/>
+        <parent link="base_link"/>
+        <child link="pillar_link"/>
+    </joint>
+    <link name="pillar_link">
         <visual>
-            <origin xyz="0 0 ${stem_length/2}" rpy="0 0 0"/>
+            <origin xyz="0 0 ${platform_height / 2}" rpy="0 0 0"/>
             <geometry>
-                <cylinder length="${stem_length}" radius="0.1" />
+                <cylinder length="${platform_height}" radius="0.1" />
             </geometry>
             <material name="grey"/>
         </visual>
     </link>
+    <joint name="platform_joint" type="revolute">
+        <origin xyz="0 0 ${platform_height + .05}" rpy="0 0 0"/>
+        <parent link="pillar_link"/>
+        <child link="platform_link"/>
+        <axis xyz="0 1 0"/>
+        <limit lower="0" upper="${pi/4}" velocity="100" effort="100"/>
+    </joint>
+    <link name="platform_link">
+    <visual>
+        <origin xyz="0 0 0" rpy="0 0 0"/>
+        <geometry>
+            <cylinder length=".1" radius="${platform_radius}" />
+        </geometry>
+        <material name="yellow"/>
+    </visual>
+    </link>
+    <!-- <joint name="stem_joint" type="revolute">
+        <origin xyz="0 0 -.25" rpy="0 0 0"/>
+        <parent link="base_link"/>
+        <child link="stem_link"/>
+        <axis xyz="0 0 1"/>
+    </joint>
+    <link name="stem_link">
+        <visual>
+            <origin xyz="0 0 -.25" rpy="${pi/2} 0 0"/>
+            <geometry>
+                <cylinder length=".2" radius="0.1" />
+            </geometry>
+            <material name="purple"/>
+        </visual>
+    </link> -->
 </robot>

File: turtle_brick/urdf/usefulstuff.xacro (robot description, xacro)
@@ -2,5 +2,5 @@
 <robot xmlns:xacro="http://www.ros.org/wiki/xacro" >
     <!-- Specify some colours -->
-    <material name="green">
+    <material name="grey">
         <color rgba=".6 .6 .6 1"/>
     </material>
@@ -11,3 +11,6 @@
         <color rgba="1 1 0 1"/>
     </material>
+    <material name="purple">
+        <color rgba="1 0 1 1"/>
+    </material>
 </robot>

Commit message: my beautiful robot

File: turtle_brick/urdf/turtle_bot.urdf (robot description, URDF)
Before this commit: robot turtlebot, 4 links, 3 joints
Links:
- added link stem_link; visual cylinder length=.2 radius=0.2
- added link wheel_link; visual cylinder length=.2 radius=0.5
Joints:
- added joint stem_joint: type revolute, parent base_link, child stem_link, origin xyz=0 0 -.25 rpy=0 0 0, axis 0 0 1, limit lower=-3.141592653589793 upper=3.141592653589793 effort=100 velocity=100
- added joint wheel_joint: type revolute, parent stem_link, child wheel_link, origin xyz=0 0 -0.7 rpy=0 0 0, axis 0 1 0, limit lower=-3.141592653589793 upper=3.141592653589793 effort=100 velocity=100

File: turtle_brick/urdf/turtle_bot.urdf.xacro (robot description, xacro)
@@ -50,18 +50,35 @@
     </visual>
     </link>
-    <!-- <joint name="stem_joint" type="revolute">
+    <joint name="stem_joint" type="revolute">
         <origin xyz="0 0 -.25" rpy="0 0 0"/>
         <parent link="base_link"/>
         <child link="stem_link"/>
         <axis xyz="0 0 1"/>
+        <limit lower="${-1*pi}" upper="${pi}" velocity="100" effort="100"/>
     </joint>
     <link name="stem_link">
         <visual>
-            <origin xyz="0 0 -.25" rpy="${pi/2} 0 0"/>
+            <origin xyz="0 0 -.1" rpy="${pi} 0 0"/>
             <geometry>
-                <cylinder length=".2" radius="0.1" />
+                <cylinder length=".2" radius="0.2" />
             </geometry>
             <material name="purple"/>
         </visual>
-    </link> -->
+    </link>
+    <joint name="wheel_joint" type="revolute">
+        <origin xyz="0 0 ${-1*wheel_radius-.2}" rpy="0 0 0"/>
+        <parent link="stem_link"/>
+        <child link="wheel_link"/>
+        <axis xyz="0 1 0"/>
+        <limit lower="${-1*pi}" upper="${pi}" velocity="100" effort="100"/>
+    </joint>
+    <link name="wheel_link">
+        <visual>
+            <origin xyz="0 0 0" rpy="${pi/2} 0 0"/>
+            <geometry>
+                <cylinder length=".2" radius="${wheel_radius}" />
+            </geometry>
+            <material name="purple"/>
+        </visual>
+    </link>
 </robot>

Commit message: Robot moves when controlled via cmd_vel

File: turtle_brick/urdf/turtle_bot.urdf (robot description, URDF)
Before this commit: robot turtlebot, 6 links, 5 joints
Links:
- removed link world
Joints:
- removed joint base_joint

File: turtle_brick/urdf/turtle_bot.urdf.xacro (robot description, xacro)
@@ -5,24 +5,18 @@
     <xacro:property name="platform_radius" value="1" />
     <xacro:property name="wheel_radius" value="0.5" />
-    <link name="world"></link>
-        <joint name="base_joint" type="fixed">
+    <link name="base_link">
+        <visual>
             <origin xyz="0 0 0" rpy="0 0 0"/>
-            <parent link="world"/>
-            <child link="base_link"/>
-        </joint>
-        <link name="base_link">
-            <visual>
-                <origin xyz="0 0 0" rpy="0 0 0"/>
-                <geometry>
-                    <box size="1 1 .5" />
-                </geometry>
-                <material name="cyan"/>
-            </visual>
-        </link>
-        <joint name="pillar_joint" type="fixed">
-            <origin xyz="0 0 .25" rpy="0 0 0"/>
-            <parent link="base_link"/>
-            <child link="pillar_link"/>
-        </joint>
+            <geometry>
+                <box size="1 1 .5" />
+            </geometry>
+            <material name="cyan"/>
+        </visual>
+    </link>
+    <joint name="pillar_joint" type="fixed">
+        <origin xyz="0 0 .25" rpy="0 0 0"/>
+        <parent link="base_link"/>
+        <child link="pillar_link"/>
+    </joint>
     <link name="pillar_link">
         <visual>

Commit message: citations + updates

File: turtle_brick/urdf/turtle_bot.urdf (robot description, URDF)
Before this commit: robot turtlebot, 5 links, 4 joints
Links:
- link pillar_link: geometry visual cylinder length=2 radius=0.1
- link wheel_link: geometry visual cylinder length=.2 radius=0.1
Joints:
- joint platform_joint: origin xyz=0 0 1.05 rpy=0 0 0 -> xyz=0 0 2.05 rpy=0 0 0
- joint wheel_joint: origin xyz=0 0 -0.7 rpy=0 0 0 -> xyz=0 0 -0.30000000000000004 rpy=0 0 0

File: turtle_brick/urdf/turtle_bot.urdf.xacro (robot description, xacro)
@@ -1,8 +1,12 @@
 <?xml version="1.0"?>
 <robot xmlns:xacro="http://www.ros.org/wiki/xacro"  name="turtlebot">
-    <xacro:include filename="usefulstuff.xacro" />
-    <xacro:property name="platform_height" value="1" />
+    <xacro:include filename="$(find turtle_brick)/usefulstuff.xacro" />
+    <!-- ########## Begin_Citation[1] ##########-->
+    <xacro:property name="yaml" value="$(find turtle_brick)/turtle.yaml" />
+    <xacro:property name="config" value="${xacro.load_yaml(yaml)}"/>
     <xacro:property name="platform_radius" value="1" />
-    <xacro:property name="wheel_radius" value="0.5" />
+    <xacro:property name="platform_height" value="${config['platform_height']}" />
+    <xacro:property name="wheel_radius" value="${config['wheel_radius']}" />
+    <!-- ########## End_Citation[1] ##########-->
     <link name="base_link">
         <visual>

Commit message: Approximately properly set up launchfiles

File: turtle_brick/urdf/turtle_bot.urdf (robot description, URDF)
Before this commit: robot turtlebot, 5 links, 4 joints
Links:
- link pillar_link: geometry visual cylinder length=1 radius=0.1
- link wheel_link: geometry visual cylinder length=.2 radius=1
Joints:
- joint platform_joint: origin xyz=0 0 2.05 rpy=0 0 0 -> xyz=0 0 1.05 rpy=0 0 0
- joint stem_joint: limit lower=-3.141592653589793 upper=3.141592653589793 effort=100 velocity=100 -> (none); type revolute -> continuous
- joint wheel_joint: limit lower=-3.141592653589793 upper=3.141592653589793 effort=100 velocity=100 -> (none); origin xyz=0 0 -0.30000000000000004 rpy=0 0 0 -> xyz=0 0 -1.2 rpy=0 0 0; type revolute -> continuous

File: turtle_brick/urdf/turtle_bot.urdf.xacro (robot description, xacro)
@@ -1,11 +1,13 @@
-<?xml version="1.0"?>
 <robot xmlns:xacro="http://www.ros.org/wiki/xacro"  name="turtlebot">
-    <xacro:include filename="$(find turtle_brick)/usefulstuff.xacro" />
+    <!-- <xacro:include filename="$(find turtle_brick)/usefulstuff.xacro" /> -->
+    <xacro:include filename="usefulstuff.xacro" />
     <!-- ########## Begin_Citation[1] ##########-->
     <xacro:property name="yaml" value="$(find turtle_brick)/turtle.yaml" />
     <xacro:property name="config" value="${xacro.load_yaml(yaml)}"/>
     <xacro:property name="platform_radius" value="1" />
-    <xacro:property name="platform_height" value="${config['platform_height']}" />
-    <xacro:property name="wheel_radius" value="${config['wheel_radius']}" />
+    <!-- <xacro:property name="platform_height" value="${config['platform_height']}" />
+    <xacro:property name="wheel_radius" value="${config['wheel_radius']}" /> -->
+        <xacro:property name="platform_height" value="1" />
+    <xacro:property name="wheel_radius" value="$1" />
     <!-- ########## End_Citation[1] ##########-->
     <link name="base_link">
@@ -32,10 +34,9 @@
         </visual>
     </link>
-    <joint name="platform_joint" type="revolute">
+    <joint name="platform_joint" type="continuous">
         <origin xyz="0 0 ${platform_height + .05}" rpy="0 0 0"/>
         <parent link="pillar_link"/>
         <child link="platform_link"/>
         <axis xyz="0 1 0"/>
-        <limit lower="0" upper="${pi/4}" velocity="100" effort="100"/>
     </joint>
     <link name="platform_link">
@@ -48,10 +49,9 @@
     </visual>
     </link>
-    <joint name="stem_joint" type="revolute">
+    <joint name="stem_joint" type="continuous">
         <origin xyz="0 0 -.25" rpy="0 0 0"/>
         <parent link="base_link"/>
         <child link="stem_link"/>
         <axis xyz="0 0 1"/>
-        <limit lower="${-1*pi}" upper="${pi}" velocity="100" effort="100"/>
     </joint>
     <link name="stem_link">
