Commit message: Loading from config in a test file

File: turtle_brick/urdf/test.urdf.xacro (robot description, xacro)
@@ -1,14 +1,9 @@
 <robot xmlns:xacro="http://www.ros.org/wiki/xacro"  name="turtlebot">
     <xacro:include filename="$(find turtle_brick)/usefulstuff.xacro" />
-    <!-- <xacro:include filename="usefulstuff.xacro" /> -->
-    <!-- ########## Begin_Citation[1] ##########-->
     <xacro:property name="yaml" value="$(find turtle_brick)/turtle.yaml" />
     <xacro:property name="config" value="${xacro.load_yaml(yaml)}"/>
-    <xacro:property name="platform_radius" value="1" />
     <xacro:property name="platform_height" value="${config['platform_height']}" />
     <xacro:property name="wheel_radius" value="${config['wheel_radius']}" />
-    <!-- <xacro:property name="platform_height" value="1" />
-    <xacro:property name="wheel_radius" value="1" /> -->
-    <!-- ########## End_Citation[1] ##########-->
+    <xacro:property name="platform_radius" value="1" />
     <link name="base_link">
         <visual>
