Commit message: little tweaks to ze bot

File: turtle_brick/urdf/turtle_bot.urdf.xacro (robot description, xacro)
@@ -6,23 +6,23 @@
     <xacro:property name="wheel_radius" value="0.5" />
     <link name="world"></link>
-    <joint name="base_joint" type="fixed">
-        <origin xyz="0 0 0" rpy="0 0 0"/>
-        <parent link="world"/>
-        <child link="base_link"/>
-    </joint>
-    <link name="base_link">
-        <visual>
+        <joint name="base_joint" type="fixed">
             <origin xyz="0 0 0" rpy="0 0 0"/>
-            <geometry>
-                <box size="1 1 .5" />
-            </geometry>
-            <material name="cyan"/>
-        </visual>
-    </link>
-    <joint name="pillar_joint" type="fixed">
-        <origin xyz="0 0 .25" rpy="0 0 0"/>
-        <parent link="base_link"/>
-        <child link="pillar_link"/>
-    </joint>
+            <parent link="world"/>
+            <child link="base_link"/>
+        </joint>
+        <link name="base_link">
+            <visual>
+                <origin xyz="0 0 0" rpy="0 0 0"/>
+                <geometry>
+                    <box size="1 1 .5" />
+                </geometry>
+                <material name="cyan"/>
+            </visual>
+        </link>
+        <joint name="pillar_joint" type="fixed">
+            <origin xyz="0 0 .25" rpy="0 0 0"/>
+            <parent link="base_link"/>
+            <child link="pillar_link"/>
+        </joint>
     <link name="pillar_link">
         <visual>

Commit message: internal joint state publisher

File: turtle_brick/urdf/turtle_bot.urdf.xacro (robot description, xacro)
@@ -59,10 +59,9 @@
         </visual>
     </link>
-    <joint name="wheel_joint" type="revolute">
+    <joint name="wheel_joint" type="continuous">
         <origin xyz="0 0 ${-1 * wheel_radius -0.2}" rpy="0 0 0"/>
         <parent link="stem_link"/>
         <child link="wheel_link"/>
         <axis xyz="0 1 0"/>
-        <limit lower="${-1*pi}" upper="${pi}" velocity="100" effort="100"/>
     </joint>
     <link name="wheel_link">

Commit message: Death to xacro for this

File: turtle_brick/urdf/turtle_bot.urdf.xacro (robot description, xacro)
@@ -1,9 +1,13 @@
 <robot xmlns:xacro="http://www.ros.org/wiki/xacro"  name="turtlebot">
     <xacro:include filename="$(find turtle_brick)/usefulstuff.xacro" />
+    <!-- Begin_Citation[1] -->
     <xacro:property name="yaml" value="$(find turtle_brick)/turtle.yaml" />
-    <xacro:property name="config" value="${xacro.load_yaml(yaml)}"/>
+    <!-- Begin_Citation[2] -->
+    <xacro:property name="config" value="${xacro.load_yaml(yaml)['/**']['ros__parameters']}"/>
+    <!-- End_Citation[2] -->
     <xacro:property name="platform_height" value="${config['platform_height']}" />
     <xacro:property name="wheel_radius" value="${config['wheel_radius']}" />
     <xacro:property name="platform_radius" value="1" />
+    <!-- End_Citation[1] -->
     <link name="base_link">
         <visual>

Commit message: uhgughughughguhgu

File: turtle_brick/urdf/turtle_bot.urdf.xacro (robot description, xacro)
@@ -26,7 +26,7 @@
     <link name="pillar_link">
         <visual>
-            <origin xyz="0 0 ${platform_height / 2}" rpy="0 0 0"/>
+            <origin xyz="0 0 ${(platform_height - ((2 * wheel_radius) + .5 + .2)) / 2}" rpy="0 0 0"/>
             <geometry>
-                <cylinder length="${platform_height}" radius="0.1" />
+                <cylinder length="${platform_height - ((2 * wheel_radius) + .5 + .2)}" radius="0.1" />
             </geometry>
             <material name="grey"/>
@@ -34,5 +34,5 @@
     </link>
     <joint name="platform_joint" type="continuous">
-        <origin xyz="0 0 ${platform_height + .05}" rpy="0 0 0"/>
+        <origin xyz="0 0 ${platform_height - ((2 * wheel_radius) + .5 + .2) + .05}" rpy="0 0 0"/>
         <parent link="pillar_link"/>
         <child link="platform_link"/>

Commit message: DRY!!!

File: turtle_brick/urdf/turtle_bot.urdf.xacro (robot description, xacro)
@@ -10,4 +10,5 @@
     <xacro:property name="platform_radius" value="1" />
     <!-- End_Citation[1] -->
+    <xacro:property name="platform_offset" value="${platform_height - ((2 * wheel_radius) + .5 + .2)}" />
     <link name="base_link">
         <visual>
@@ -26,7 +27,7 @@
     <link name="pillar_link">
         <visual>
-            <origin xyz="0 0 ${(platform_height - ((2 * wheel_radius) + .5 + .2)) / 2}" rpy="0 0 0"/>
+            <origin xyz="0 0 ${platform_offset / 2}" rpy="0 0 0"/>
             <geometry>
-                <cylinder length="${platform_height - ((2 * wheel_radius) + .5 + .2)}" radius="0.1" />
+                <cylinder length="${platform_offset}" radius="0.1" />
             </geometry>
             <material name="grey"/>
@@ -34,5 +35,5 @@
     </link>
     <joint name="platform_joint" type="continuous">
-        <origin xyz="0 0 ${platform_height - ((2 * wheel_radius) + .5 + .2) + .05}" rpy="0 0 0"/>
+        <origin xyz="0 0 ${platform_offset + .05}" rpy="0 0 0"/>
         <parent link="pillar_link"/>
         <child link="platform_link"/>
